File: hardware/weatherMat.brd (EAGLE design)
At the start: 162.7 x 112.7 mm, 29 parts, among them IC1 MCP3008, IC2 LM2596S, J1 MAGJACK, J2 RASPBERRYPI-40-PIN-GPIOJIM, J3 Air Digitals, J4 Soil Temp, J5 Air Analogs, J6 RJ11, J7 RJ11, U1 MAGJACK-POE

Commit message: Update
Parts:
- moved U$1 29.2 mm to (186.7, 42.4)
- moved U$2 12.7 mm to (-32.6, -16.0)
- moved L1 8.65 mm to (86.7, 31.5)
- moved C3 7.23 mm to (47.4, 50.9), turned to 90 degrees
- moved J3 5.08 mm to (85.3, 75.2)
- moved C2 5.08 mm to (39.4, 47.8)
- moved C4 5.08 mm to (35.7, 21.6)
- moved C5 5.08 mm to (61.3, 20.6)
- moved D2 5.08 mm to (60.6, 37.6)
- moved R2 5.08 mm to (30.1, 43.3)
- moved R3 5.08 mm to (30.1, 52.3)
- moved R4 5.08 mm to (30.1, 47.9)
- moved U1 5.08 mm to (31.1, 6.86)
- moved J1 5.08 mm to (-4.83, 50.0)
- moved J6 5.08 mm to (4.06, 62.7)
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Routing:
- net GP6: track 117.9 -> 60.1 mm, vias 0 -> 1
- net +3V3: track 222.5 -> 180.9 mm, vias 0 -> 1
- net N$6: track 47.4 -> 60.7 mm
- net N$15: track 38.8 -> 26.9 mm, vias 0 -> 1
- net N$16: track 51.1 -> 40.2 mm
- net +5V: track 131.8 -> 142.1 mm
- net N$14: track 49.5 -> 57.0 mm
- net N$18: track 60.3 -> 52.8 mm, vias 0 -> 1
- net N$3: track 42.9 -> 47.4 mm
- net GP5: track 49.8 -> 45.4 mm
- net N$19: track 59.8 -> 55.9 mm, vias 0 -> 1
- net N$2: track 14.5 -> 12.4 mm
- net N$1: track 58.2 -> 56.6 mm
- net N$5: track 53.5 -> 52.3 mm
- net N$12: track 60.8 -> 61.7 mm
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- added copper zone on layer 1, net GND
Other:
- board text added: "PolyCase WC-24F"
- board text added: "Routable area for Eagle freeware is 4" x 3.2""

Commit message: Update
Parts:
- removed U$1: (no value), Jims:PIOUTLINE
Changed lines of the file:
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@@
 </element>
 <element name="U$2" library="Jims" package="WC-24F" value="" x="-32.639" y="-16.002"/>
-<element name="U$1" library="Jims" package="PIOUTLINE" value="" x="186.69" y="42.418"/>
 <element name="C1" library="SparkFun-Capacitors" package="CAP-PTH-SMALL" value="0.1uF" x="19.431" y="14.859" smashed="yes" rot="R90">
 <attribute name="NAME" x="18.034" y="14.859" size="0.8128" layer="25" font="vector" ratio="12" rot="R180"/>

Commit message: Updates
Parts:
- moved J3 7.47 mm to (77.9, 75.3)
- moved J4 5.51 mm to (68.2, 0.58)
Routing:
- net N$6: track 60.7 -> 46.6 mm
- net N$16: track 40.2 -> 50.9 mm
- net N$17: track 49.8 -> 40.1 mm, vias 0 -> 1
- net +5V: track 142.1 -> 133.1 mm
- net N$15: track 26.9 -> 34.3 mm
- net N$18: track 52.8 -> 46.7 mm
- net GP12_DHT: track 35.4 -> 29.9 mm
- net N$21: track 65.4 -> 70.7 mm
- net +3V3: track 180.9 -> 185.4 mm, vias 1 -> 0
- net N$12: track 61.7 -> 58.4 mm
- net N$20: track 59.1 -> 61.7 mm
- net N$3: track 47.4 -> 49.8 mm
- net N$5: track 52.3 -> 50.1 mm
- net GP6: track 60.1 -> 61.2 mm
- net N$4: track 50.7 -> 51.3 mm

Commit message: Board update
Parts:
- moved D1 19.9 mm to (77.1, 12.4), turned to 180 degrees
- moved C5 14.7 mm to (48.2, 14.0), turned to 90 degrees
- moved C6 8.63 mm to (64.9, 25.2)
- moved IC2 1.59 mm to (46.2, 26.0)
Routing:
- net N$14: track 57.0 -> 42.9 mm
- net V+: track 31.5 -> 22.2 mm
- net N$1: track 56.6 -> 48.4 mm
- net +3V3: track 185.4 -> 177.7 mm
- net +5V: track 133.1 -> 129.2 mm
- net N$4: track 51.3 -> 50.6 mm
Other:
- board text removed: "Routable area for Eagle freeware is 4" x 3.2""

Commit message: board updates
Connections:
- removed net N$19: IC1.4, J5.4
- net GND: now also IC1.2, IC1.4, IC1.6, IC1.7, IC1.8
- net N$17: now also IC1.3; no longer IC1.2
- net N$18: now also IC1.5; no longer IC1.3
Routing:
- net N$19: track 56.3 -> 0.00 mm, vias 1 -> 0
- net +3V3: track 177.7 -> 163.2 mm
- net N$18: track 46.7 -> 51.8 mm
- net N$17: track 40.1 -> 42.6 mm
- net GP6: track 61.2 -> 60.1 mm
Changed lines of the file:
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@@
 <vertex x="130.81" y="-16.51"/>
 </polygon>
+<contactref element="IC1" pad="8"/>
+<contactref element="IC1" pad="6"/>
+<contactref element="IC1" pad="7"/>
+<contactref element="IC1" pad="4"/>
+<contactref element="IC1" pad="2"/>
 <wire x1="78.867" y1="61.849" x2="73.787" y2="64.389" width="0" layer="19" extent="1-1"/>
 </signal>
@@
 <contactref element="J4" pad="1"/>
 <wire x1="56.007" y1="55.88" x2="53.467" y2="55.88" width="1.016" layer="1"/>
-<wire x1="56.134" y1="59.944" x2="56.134" y2="55.88" width="1.016" layer="16"/>
-<wire x1="66.802" y1="59.944" x2="56.134" y2="59.944" width="1.016" layer="16"/>
-<wire x1="68.707" y1="61.849" x2="67.056" y2="60.198" width="1.016" layer="16"/>
-<wire x1="67.056" y1="60.198" x2="66.802" y2="59.944" width="1.016" layer="16"/>
-<wire x1="56.134" y1="55.88" x2="56.007" y2="55.88" width="1.016" layer="16"/>
-<wire x1="47.498" y1="48.514" x2="47.498" y2="50.8" width="1.016" layer="1"/>
-<wire x1="48.514" y1="47.498" x2="47.498" y2="48.514" width="1.016" layer="1"/>
-<wire x1="52.07" y1="47.498" x2="48.514" y2="47.498" width="1.016" layer="1"/>
-<wire x1="52.07" y1="54.61" x2="52.07" y2="47.498" width="1.016" layer="1"/>
-<wire x1="53.086" y1="55.626" x2="52.07" y2="54.61" width="1.016" layer="1"/>
-<wire x1="47.498" y1="50.8" x2="47.371" y2="50.927" width="1.016" layer="1"/>
+<wire x1="48.514" y1="51.054" x2="53.086" y2="55.626" width="1.016" layer="1"/>
+<wire x1="47.498" y1="51.054" x2="48.514" y2="51.054" width="1.016" layer="1"/>
 <wire x1="53.086" y1="55.626" x2="53.467" y2="55.88" width="1.016" layer="1"/>
+<wire x1="47.498" y1="51.054" x2="47.371" y2="50.927" width="1.016" layer="1"/>
+<wire x1="64.77" y1="57.912" x2="67.056" y2="60.198" width="1.016" layer="16"/>
+<wire x1="67.056" y1="60.198" x2="68.707" y2="61.849" width="1.016" layer="16"/>
+<wire x1="57.912" y1="57.912" x2="64.77" y2="57.912" width="1.016" layer="16"/>
+<wire x1="55.88" y1="55.88" x2="57.912" y2="57.912" width="1.016" layer="16"/>
+<wire x1="55.88" y1="55.88" x2="56.007" y2="55.88" width="1.016" layer="16"/>
 <wire x1="87.122" y1="59.944" x2="89.027" y2="61.849" width="1.016" layer="16"/>
 <wire x1="67.31" y1="59.944" x2="87.122" y2="59.944" width="1.016" layer="16"/>
@@
 <wire x1="31.242" y1="19.812" x2="49.022" y2="19.812" width="1.016" layer="16"/>
 <wire x1="29.464" y1="21.59" x2="31.242" y2="19.812" width="1.016" layer="16"/>
-<wire x1="49.784" y1="59.436" x2="53.34" y2="55.88" width="1.016" layer="16"/>
-<wire x1="29.718" y1="59.436" x2="49.784" y2="59.436" width="1.016" layer="16"/>
-<wire x1="53.34" y1="55.88" x2="53.467" y2="55.88" width="1.016" layer="16"/>
+<wire x1="41.402" y1="56.896" x2="47.371" y2="50.927" width="1.016" layer="16"/>
+<wire x1="32.258" y1="56.896" x2="41.402" y2="56.896" width="1.016" layer="16"/>
+<wire x1="29.718" y1="59.436" x2="32.258" y2="56.896" width="1.016" layer="16"/>
 </signal>
 <signal name="N$14" class="1">
@@
 <wire x1="19.304" y1="21.59" x2="12.954" y2="21.59" width="0.3048" layer="1"/>
 <wire x1="12.954" y1="21.59" x2="12.954" y2="21.717" width="0.3048" layer="1"/>
-<wire x1="48.768" y1="59.69" x2="50.927" y2="61.849" width="0.3048" layer="1"/>
-<wire x1="48.768" y1="48.768" x2="48.768" y2="59.69" width="0.3048" layer="1"/>
-<wire x1="21.59" y1="21.59" x2="48.768" y2="48.768" width="0.3048" layer="16"/>
-<wire x1="19.304" y1="21.59" x2="21.59" y2="21.59" width="0.3048" layer="16"/>
-<via x="48.768" y="48.768" extent="1-16" drill="0.3302"/>
+<wire x1="40.64" y1="51.562" x2="50.927" y2="61.849" width="0.3048" layer="1"/>
+<wire x1="40.64" y1="42.418" x2="40.64" y2="51.562" width="0.3048" layer="1"/>
+<wire x1="19.812" y1="21.59" x2="40.64" y2="42.418" width="0.3048" layer="16"/>
+<wire x1="19.304" y1="21.59" x2="19.812" y2="21.59" width="0.3048" layer="16"/>
+<via x="40.64" y="42.418" extent="1-16" drill="0.3302"/>
 </signal>
 <signal name="N$13">
@@
 <wire x1="19.558" y1="59.436" x2="14.224" y2="59.436" width="0.3048" layer="16"/>
 <wire x1="12.954" y1="60.706" x2="12.954" y2="60.833" width="0.3048" layer="16"/>
-</signal>
-<signal name="N$17">
-<contactref element="IC1" pad="2"/>
-<contactref element="J5" pad="2"/>
-<wire x1="51.562" y1="52.578" x2="55.88" y2="48.26" width="0.3048" layer="16"/>
-<wire x1="50.038" y1="52.578" x2="51.562" y2="52.578" width="0.3048" layer="16"/>
-<wire x1="46.228" y1="56.388" x2="50.038" y2="52.578" width="0.3048" layer="16"/>
-<wire x1="44.196" y1="56.388" x2="46.228" y2="56.388" width="0.3048" layer="16"/>
-<wire x1="37.846" y1="62.738" x2="44.196" y2="56.388" width="0.3048" layer="1"/>
-<wire x1="37.846" y1="67.31" x2="37.846" y2="62.738" width="0.3048" layer="1"/>
-<wire x1="29.972" y1="75.184" x2="37.846" y2="67.31" width="0.3048" layer="1"/>
-<wire x1="55.88" y1="48.26" x2="56.007" y2="48.26" width="0.3048" layer="16"/>
-<wire x1="29.972" y1="75.184" x2="29.774" y2="75.184" width="0.3048" layer="1"/>
-<via x="44.196" y="56.388" extent="1-16" drill="0.3302"/>
-</signal>
-<signal name="N$18">
-<contactref element="IC1" pad="3"/>
-<contactref element="J5" pad="3"/>
-<wire x1="53.34" y1="53.34" x2="58.42" y2="48.26" width="0.3048" layer="16"/>
-<wire x1="50.038" y1="53.34" x2="53.34" y2="53.34" width="0.3048" layer="16"/>
-<wire x1="46.228" y1="57.15" x2="50.038" y2="53.34" width="0.3048" layer="16"/>
-<wire x1="38.862" y1="57.15" x2="46.228" y2="57.15" width="0.3048" layer="16"/>
-<wire x1="31.242" y1="64.77" x2="38.862" y2="57.15" width="0.3048" layer="1"/>
-<wire x1="31.242" y1="70.358" x2="31.242" y2="64.77" width="0.3048" layer="1"/>
-<wire x1="26.416" y1="75.184" x2="31.242" y2="70.358" width="0.3048" layer="1"/>
-<wire x1="58.42" y1="48.26" x2="58.547" y2="48.26" width="0.3048" layer="16"/>
-<wire x1="26.416" y1="75.184" x2="26.274" y2="75.184" width="0.3048" layer="1"/>
-<via x="38.862" y="57.15" extent="1-16" drill="0.3302"/>
-</signal>
-<signal name="N$19">
-<contactref element="IC1" pad="4"/>
-<contactref element="J5" pad="4"/>
-<wire x1="55.118" y1="54.102" x2="60.96" y2="48.26" width="0.3048" layer="16"/>
-<wire x1="51.054" y1="54.102" x2="55.118" y2="54.102" width="0.3048" layer="16"/>
-<wire x1="47.244" y1="57.912" x2="51.054" y2="54.102" width="0.3048" layer="16"/>
-<wire x1="28.448" y1="57.912" x2="47.244" y2="57.912" width="0.3048" layer="16"/>
-<wire x1="22.86" y1="63.5" x2="28.448" y2="57.912" width="0.3048" layer="1"/>
-<wire x1="22.86" y1="75.184" x2="22.86" y2="63.5" width="0.3048" layer="1"/>
-<wire x1="60.96" y1="48.26" x2="61.087" y2="48.26" width="0.3048" layer="16"/>
-<wire x1="22.86" y1="75.184" x2="22.774" y2="75.184" width="0.3048" layer="1"/>
-<via x="28.448" y="57.912" extent="1-16" drill="0.3302"/>
 </signal>
 <signal name="N$15">
@@
 <wire x1="75.438" y1="0.762" x2="75.2498" y2="0.5842" width="0.3048" layer="1"/>
 </signal>
+<signal name="N$17">
+<contactref element="IC1" pad="3"/>
+<contactref element="J5" pad="2"/>
+<wire x1="53.34" y1="53.34" x2="58.42" y2="48.26" width="0.3048" layer="16"/>
+<wire x1="49.276" y1="53.34" x2="53.34" y2="53.34" width="0.3048" layer="16"/>
+<wire x1="45.212" y1="57.404" x2="49.276" y2="53.34" width="0.3048" layer="16"/>
+<wire x1="43.18" y1="57.404" x2="45.212" y2="57.404" width="0.3048" layer="16"/>
+<wire x1="37.846" y1="62.738" x2="43.18" y2="57.404" width="0.3048" layer="1"/>
+<wire x1="37.846" y1="67.31" x2="37.846" y2="62.738" width="0.3048" layer="1"/>
+<wire x1="29.972" y1="75.184" x2="37.846" y2="67.31" width="0.3048" layer="1"/>
+<wire x1="58.42" y1="48.26" x2="58.547" y2="48.26" width="0.3048" layer="16"/>
+<wire x1="29.972" y1="75.184" x2="29.774" y2="75.184" width="0.3048" layer="1"/>
+<via x="43.18" y="57.404" extent="1-16" drill="0.3302"/>
+</signal>
+<signal name="N$18">
+<contactref element="IC1" pad="5"/>
+<contactref element="J5" pad="3"/>
+<wire x1="57.658" y1="54.102" x2="63.5" y2="48.26" width="0.3048" layer="16"/>
+<wire x1="49.276" y1="54.102" x2="57.658" y2="54.102" width="0.3048" layer="16"/>
+<wire x1="45.212" y1="58.166" x2="49.276" y2="54.102" width="0.3048" layer="16"/>
+<wire x1="37.846" y1="58.166" x2="45.212" y2="58.166" width="0.3048" layer="16"/>
+<wire x1="31.242" y1="64.77" x2="37.846" y2="58.166" width="0.3048" layer="1"/>
+<wire x1="31.242" y1="70.358" x2="31.242" y2="64.77" width="0.3048" layer="1"/>
+<wire x1="26.416" y1="75.184" x2="31.242" y2="70.358" width="0.3048" layer="1"/>
+<wire x1="63.5" y1="48.26" x2="63.627" y2="48.26" width="0.3048" layer="16"/>
+<wire x1="26.416" y1="75.184" x2="26.274" y2="75.184" width="0.3048" layer="1"/>
+<via x="37.846" y="58.166" extent="1-16" drill="0.3302"/>
+</signal>
 </signals>
