File: hardware/weatherMat.sch (EAGLE design)
At the start: 27 parts, among them IC1 MCP3008, IC2 LM2596S, J1 MAGJACK, J2 RASPBERRYPI-40-PIN-GPIOJIM, J3 Air Digitals, J4 Soil Temp, J5 Air Analogs, J6 RJ11, J7 RJ11, U1 MAGJACK-POE

Commit message: board updates
Connections:
- removed net N$19: IC1.CH3, J5.4
- net GND: now also IC1.CH1, IC1.CH3, IC1.CH5, IC1.CH6, IC1.CH7
- net N$17: now also IC1.CH2; no longer IC1.CH1
- net N$18: now also IC1.CH4; no longer IC1.CH2
Changed lines of the file:
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@@
 <part name="C1" library="SparkFun-Capacitors" deviceset="CAP" device="PTH" value="0.1uF"/>
 <part name="GND4" library="SparkFun-Aesthetics" deviceset="GND" device=""/>
+<part name="GND12" library="SparkFun-Aesthetics" deviceset="GND" device=""/>
 </parts>
 <sheets>
@@
 </instance>
 <instance part="GND4" gate="1" x="68.58" y="53.34"/>
+<instance part="GND12" gate="1" x="134.62" y="-35.56"/>
 </instances>
 <busses>
@@
 <wire x1="68.58" y1="55.88" x2="68.58" y2="58.42" width="0.1524" layer="91"/>
 </segment>
+<segment>
+<pinref part="IC1" gate="G$1" pin="CH7"/>
+<pinref part="GND12" gate="1" pin="GND"/>
+<wire x1="132.08" y1="-25.4" x2="134.62" y2="-25.4" width="0.1524" layer="91"/>
+<wire x1="134.62" y1="-25.4" x2="134.62" y2="-33.02" width="0.1524" layer="91"/>
+<pinref part="IC1" gate="G$1" pin="CH5"/>
+<wire x1="132.08" y1="-20.32" x2="134.62" y2="-20.32" width="0.1524" layer="91"/>
+<wire x1="134.62" y1="-20.32" x2="134.62" y2="-22.86" width="0.1524" layer="91"/>
+<junction x="134.62" y="-25.4"/>
+<pinref part="IC1" gate="G$1" pin="CH6"/>
+<wire x1="134.62" y1="-22.86" x2="134.62" y2="-25.4" width="0.1524" layer="91"/>
+<wire x1="132.08" y1="-22.86" x2="134.62" y2="-22.86" width="0.1524" layer="91"/>
+<junction x="134.62" y="-22.86"/>
+<pinref part="IC1" gate="G$1" pin="CH3"/>
+<wire x1="132.08" y1="-15.24" x2="134.62" y2="-15.24" width="0.1524" layer="91"/>
+<wire x1="134.62" y1="-15.24" x2="134.62" y2="-20.32" width="0.1524" layer="91"/>
+<junction x="134.62" y="-20.32"/>
+<pinref part="IC1" gate="G$1" pin="CH1"/>
+<wire x1="132.08" y1="-10.16" x2="134.62" y2="-10.16" width="0.1524" layer="91"/>
+<wire x1="134.62" y1="-10.16" x2="134.62" y2="-15.24" width="0.1524" layer="91"/>
+<junction x="134.62" y="-15.24"/>
+</segment>
 </net>
 <net name="V+" class="1">
@@
 </segment>
 </net>
-<net name="N$17" class="0">
-<segment>
-<pinref part="IC1" gate="G$1" pin="CH1"/>
-<pinref part="J5" gate="G$1" pin="2"/>
-<wire x1="132.08" y1="-10.16" x2="142.24" y2="-10.16" width="0.1524" layer="91"/>
-</segment>
-</net>
-<net name="N$18" class="0">
-<segment>
-<pinref part="IC1" gate="G$1" pin="CH2"/>
-<pinref part="J5" gate="G$1" pin="3"/>
-<wire x1="132.08" y1="-12.7" x2="142.24" y2="-12.7" width="0.1524" layer="91"/>
-</segment>
-</net>
-<net name="N$19" class="0">
-<segment>
-<pinref part="IC1" gate="G$1" pin="CH3"/>
-<pinref part="J5" gate="G$1" pin="4"/>
-<wire x1="132.08" y1="-15.24" x2="142.24" y2="-15.24" width="0.1524" layer="91"/>
-</segment>
-</net>
 <net name="N$15" class="0">
 <segment>
@@
 </segment>
 </net>
+<net name="N$17" class="0">
+<segment>
+<pinref part="IC1" gate="G$1" pin="CH2"/>
+<wire x1="132.08" y1="-12.7" x2="137.16" y2="-12.7" width="0.1524" layer="91"/>
+<wire x1="137.16" y1="-12.7" x2="137.16" y2="-10.16" width="0.1524" layer="91"/>
+<pinref part="J5" gate="G$1" pin="2"/>
+<wire x1="137.16" y1="-10.16" x2="142.24" y2="-10.16" width="0.1524" layer="91"/>
+</segment>
+</net>
+<net name="N$18" class="0">
+<segment>
+<pinref part="IC1" gate="G$1" pin="CH4"/>
+<wire x1="132.08" y1="-17.78" x2="139.7" y2="-17.78" width="0.1524" layer="91"/>
+<wire x1="139.7" y1="-17.78" x2="139.7" y2="-12.7" width="0.1524" layer="91"/>
+<pinref part="J5" gate="G$1" pin="3"/>
+<wire x1="139.7" y1="-12.7" x2="142.24" y2="-12.7" width="0.1524" layer="91"/>
+</segment>
+</net>

Commit message: Updates
Other:
- note added: "Adafruit SHT10"
- note added: "Sparkfun SEN-08942"
Changed lines of the file:
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@@
 Required?</text>
 <text x="111.76" y="0" size="1.778" layer="97">8 channel ADC</text>
+<text x="203.2" y="-30.48" size="1.778" layer="97">Sparkfun SEN-08942</text>
+<text x="68.58" y="-50.8" size="1.778" layer="97">Adafruit SHT10</text>
 </plain>
 <instances>
