File: hardware/air.sch (EAGLE design)
At the start: 9 parts, among them J1 Air Digitals, J2 Air Analogs, U1 TGS2600, U2 DHT22

Commit message: board updates
Changed lines of the file:
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@@
 </instance>
 <instance part="GND4" gate="1" x="43.18" y="-7.62"/>
-<instance part="GND2" gate="1" x="-7.62" y="0"/>
+<instance part="GND2" gate="1" x="-7.62" y="7.62"/>
 <instance part="U1" gate="G$1" x="7.62" y="17.78" smashed="yes">
 <attribute name="NAME" x="5.334" y="26.162" size="1.778" layer="95"/>
@@
 <wire x1="-2.54" y1="15.24" x2="-7.62" y2="15.24" width="0.1524" layer="91"/>
 <pinref part="GND2" gate="1" pin="GND"/>
-<wire x1="-7.62" y1="15.24" x2="-7.62" y2="2.54" width="0.1524" layer="91"/>
+<wire x1="-7.62" y1="15.24" x2="-7.62" y2="10.16" width="0.1524" layer="91"/>
 <wire x1="-7.62" y1="15.24" x2="-7.62" y2="22.86" width="0.1524" layer="91"/>
 <junction x="-7.62" y="15.24"/>
@@
 <pinref part="J2" gate="G$1" pin="2"/>
 <wire x1="-25.4" y1="15.24" x2="-17.78" y2="15.24" width="0.1524" layer="91"/>
-<wire x1="-17.78" y1="15.24" x2="-17.78" y2="5.08" width="0.1524" layer="91"/>
-<wire x1="-17.78" y1="5.08" x2="20.32" y2="5.08" width="0.1524" layer="91"/>
-<wire x1="20.32" y1="5.08" x2="20.32" y2="15.24" width="0.1524" layer="91"/>
+<wire x1="-17.78" y1="15.24" x2="-17.78" y2="2.54" width="0.1524" layer="91"/>
+<wire x1="-17.78" y1="2.54" x2="20.32" y2="2.54" width="0.1524" layer="91"/>
+<wire x1="20.32" y1="2.54" x2="20.32" y2="15.24" width="0.1524" layer="91"/>
 <junction x="20.32" y="15.24"/>
 <pinref part="U1" gate="G$1" pin="2"/>

Commit message: eagle updates
Parts:
- removed R3: 10K, SparkFun-Passives:RESISTORPTH-1/4W
- removed R4: PHOTOCELLPTH, SparkFun-Sensors:PHOTOCELLPTH
- added JP2: TSL2591 Breakout, microbuilder:HEADER-1X670MIL
Connections:
- removed net N$6: J2.3, R3.1, R4.P$1
- net GND: now also JP2.2; no longer R4.P$2
- net N$1: now also JP2.1
- net N$2: now also JP2.6
- net N$8: no longer R3.2
- net SDA: now also JP2.5
Other:
- note removed: "Could this get wet with rain?"
- moved on the sheet: R1, U2

Commit message: remove light sensor from air board
Parts:
- removed JP2: TSL2591 Breakout, microbuilder:HEADER-1X670MIL
Connections:
- net GND: no longer JP2.2
- net N$1: no longer JP2.1
- net N$2: no longer JP2.6
- net SDA: no longer JP2.5
Changed lines of the file:
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@@
 <part name="GND2" library="supply1" deviceset="GND" device=""/>
 <part name="U1" library="Jims" deviceset="TGN2600" device="" value="TGS2600"/>
-<part name="JP2" library="microbuilder" deviceset="HEADER-1X6" device="70MIL" value="TSL2591 Breakout"/>
 </parts>
 <sheets>
@@
 <attribute name="VALUE" x="3.81" y="6.858" size="1.778" layer="96"/>
 </instance>
-<instance part="JP2" gate="A" x="10.16" y="76.2" rot="MR180"/>
 </instances>
 <busses>
@@
 <pinref part="J1" gate="G$1" pin="1"/>
 <pinref part="JP1" gate="A" pin="1"/>
-<wire x1="-25.4" y1="43.18" x2="0" y2="43.18" width="0.1524" layer="91"/>
-<wire x1="0" y1="43.18" x2="7.62" y2="43.18" width="0.1524" layer="91"/>
-<wire x1="0" y1="43.18" x2="0" y2="68.58" width="0.1524" layer="91"/>
-<junction x="0" y="43.18"/>
-<pinref part="JP2" gate="A" pin="1"/>
-<wire x1="0" y1="68.58" x2="7.62" y2="68.58" width="0.1524" layer="91"/>
+<wire x1="-25.4" y1="43.18" x2="7.62" y2="43.18" width="0.1524" layer="91"/>
 </segment>
 </net>
@@
 <wire x1="-7.62" y1="40.64" x2="-7.62" y2="48.26" width="0.1524" layer="91"/>
 <junction x="-7.62" y="48.26"/>
-<wire x1="-7.62" y1="53.34" x2="-7.62" y2="71.12" width="0.1524" layer="91"/>
-<junction x="-7.62" y="53.34"/>
-<pinref part="JP2" gate="A" pin="2"/>
-<wire x1="-7.62" y1="71.12" x2="7.62" y2="71.12" width="0.1524" layer="91"/>
 </segment>
 <segment>
@@
 <segment>
 <pinref part="J1" gate="G$1" pin="4"/>
-<wire x1="-25.4" y1="50.8" x2="-10.16" y2="50.8" width="0.1524" layer="91"/>
 <pinref part="JP1" gate="A" pin="4"/>
-<wire x1="-10.16" y1="50.8" x2="7.62" y2="50.8" width="0.1524" layer="91"/>
-<wire x1="-10.16" y1="50.8" x2="-10.16" y2="81.28" width="0.1524" layer="91"/>
-<junction x="-10.16" y="50.8"/>
-<pinref part="JP2" gate="A" pin="6"/>
-<wire x1="-10.16" y1="81.28" x2="7.62" y2="81.28" width="0.1524" layer="91"/>
+<wire x1="-25.4" y1="50.8" x2="7.62" y2="50.8" width="0.1524" layer="91"/>
 </segment>
 </net>
@@
 <wire x1="-25.4" y1="48.26" x2="-17.78" y2="48.26" width="0.1524" layer="91"/>
 <wire x1="-17.78" y1="48.26" x2="-17.78" y2="55.88" width="0.1524" layer="91"/>
-<wire x1="-17.78" y1="55.88" x2="-2.54" y2="55.88" width="0.1524" layer="91"/>
-<wire x1="-2.54" y1="55.88" x2="2.54" y2="55.88" width="0.1524" layer="91"/>
+<wire x1="-17.78" y1="55.88" x2="2.54" y2="55.88" width="0.1524" layer="91"/>
 <wire x1="2.54" y1="55.88" x2="2.54" y2="53.34" width="0.1524" layer="91"/>
 <pinref part="JP1" gate="A" pin="5"/>
 <wire x1="2.54" y1="53.34" x2="7.62" y2="53.34" width="0.1524" layer="91"/>
-<wire x1="-2.54" y1="55.88" x2="-2.54" y2="78.74" width="0.1524" layer="91"/>
-<junction x="-2.54" y="55.88"/>
-<pinref part="JP2" gate="A" pin="5"/>
-<wire x1="-2.54" y1="78.74" x2="7.62" y2="78.74" width="0.1524" layer="91"/>
 </segment>
 </net>

Commit message: decoupling caps
Parts:
- added C1, C2, C3: 0.1uF, SparkFun-Capacitors:CAPPTH
- R2: value 22K -> 10K
Connections:
- net 3.3V: now also C2.1
- net GND: now also C1.2, C2.2, C3.2
- net N$1: now also C3.1
- net N$8: now also C1.1
Other:
- moved on the sheet: JP1
Changed lines of the file:
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@@
 <part name="GND1" library="supply1" deviceset="GND" device=""/>
 <part name="GND3" library="supply1" deviceset="GND" device=""/>
-<part name="R2" library="SparkFun-Passives" deviceset="RESISTOR" device="PTH-1/4W" value="22K"/>
+<part name="R2" library="SparkFun-Passives" deviceset="RESISTOR" device="PTH-1/4W" value="10K"/>
 <part name="J2" library="SparkFun-Connectors" deviceset="M05" device="SCREW" value="Air Analogs"/>
 <part name="R1" library="SparkFun-Passives" deviceset="RESISTOR" device="PTH-1/4W" value="4.7K"/>
@@
 <part name="GND2" library="supply1" deviceset="GND" device=""/>
 <part name="U1" library="Jims" deviceset="TGN2600" device="" value="TGS2600"/>
+<part name="C1" library="SparkFun-Capacitors" deviceset="CAP" device="PTH" value="0.1uF"/>
+<part name="C2" library="SparkFun-Capacitors" deviceset="CAP" device="PTH" value="0.1uF"/>
+<part name="C3" library="SparkFun-Capacitors" deviceset="CAP" device="PTH" value="0.1uF"/>
 </parts>
 <sheets>
@@
 <instances>
 <instance part="U2" gate="G$1" x="45.72" y="88.9"/>
-<instance part="JP1" gate="A" x="10.16" y="48.26" rot="MR180"/>
+<instance part="JP1" gate="A" x="35.56" y="48.26" rot="MR180"/>
 <instance part="J1" gate="G$1" x="-33.02" y="48.26"/>
 <instance part="GND1" gate="1" x="-7.62" y="38.1"/>
-<instance part="GND3" gate="1" x="27.94" y="76.2"/>
+<instance part="GND3" gate="1" x="27.94" y="71.12"/>
 <instance part="R2" gate="G$1" x="25.4" y="7.62" rot="R90"/>
 <instance part="J2" gate="G$1" x="-33.02" y="17.78" smashed="yes">
@@
 <instance part="R1" gate="G$1" x="-12.7" y="99.06" rot="R90"/>
 <instance part="GND4" gate="1" x="25.4" y="-7.62"/>
-<instance part="GND2" gate="1" x="-7.62" y="7.62"/>
+<instance part="GND2" gate="1" x="-7.62" y="2.54"/>
 <instance part="U1" gate="G$1" x="7.62" y="17.78" smashed="yes">
 <attribute name="NAME" x="5.334" y="26.162" size="1.778" layer="95"/>
 <attribute name="VALUE" x="3.81" y="6.858" size="1.778" layer="96"/>
 </instance>
+<instance part="C1" gate="G$1" x="-15.24" y="12.7"/>
+<instance part="C2" gate="G$1" x="20.32" y="83.82"/>
+<instance part="C3" gate="G$1" x="12.7" y="58.42"/>
 </instances>
 <busses>
@@
 <pinref part="J1" gate="G$1" pin="1"/>
 <pinref part="JP1" gate="A" pin="1"/>
-<wire x1="-25.4" y1="43.18" x2="7.62" y2="43.18" width="0.1524" layer="91"/>
+<wire x1="-25.4" y1="43.18" x2="25.4" y2="43.18" width="0.1524" layer="91"/>
+<wire x1="25.4" y1="43.18" x2="33.02" y2="43.18" width="0.1524" layer="91"/>
+<wire x1="25.4" y1="43.18" x2="25.4" y2="66.04" width="0.1524" layer="91"/>
+<junction x="25.4" y="43.18"/>
+<wire x1="25.4" y1="66.04" x2="12.7" y2="66.04" width="0.1524" layer="91"/>
+<pinref part="C3" gate="G$1" pin="1"/>
+<wire x1="12.7" y1="66.04" x2="12.7" y2="63.5" width="0.1524" layer="91"/>
 </segment>
 </net>
@@
 <wire x1="-7.62" y1="53.34" x2="-7.62" y2="48.26" width="0.1524" layer="91"/>
 <pinref part="JP1" gate="A" pin="3"/>
-<wire x1="-7.62" y1="48.26" x2="7.62" y2="48.26" width="0.1524" layer="91"/>
+<wire x1="-7.62" y1="48.26" x2="12.7" y2="48.26" width="0.1524" layer="91"/>
 <pinref part="GND1" gate="1" pin="GND"/>
+<wire x1="12.7" y1="48.26" x2="33.02" y2="48.26" width="0.1524" layer="91"/>
 <wire x1="-7.62" y1="40.64" x2="-7.62" y2="48.26" width="0.1524" layer="91"/>
 <junction x="-7.62" y="48.26"/>
+<pinref part="C3" gate="G$1" pin="2"/>
+<wire x1="12.7" y1="48.26" x2="12.7" y2="55.88" width="0.1524" layer="91"/>
+<junction x="12.7" y="48.26"/>
 </segment>
 <segment>
@@
 <wire x1="35.56" y1="81.28" x2="27.94" y2="81.28" width="0.1524" layer="91"/>
 <pinref part="GND3" gate="1" pin="GND"/>
-<wire x1="27.94" y1="81.28" x2="27.94" y2="78.74" width="0.1524" layer="91"/>
+<wire x1="27.94" y1="81.28" x2="27.94" y2="76.2" width="0.1524" layer="91"/>
+<wire x1="27.94" y1="76.2" x2="27.94" y2="73.66" width="0.1524" layer="91"/>
+<wire x1="27.94" y1="76.2" x2="20.32" y2="76.2" width="0.1524" layer="91"/>
+<junction x="27.94" y="76.2"/>
+<pinref part="C2" gate="G$1" pin="2"/>
+<wire x1="20.32" y1="76.2" x2="20.32" y2="81.28" width="0.1524" layer="91"/>
 </segment>
 <segment>
@@
 <wire x1="-2.54" y1="15.24" x2="-7.62" y2="15.24" width="0.1524" layer="91"/>
 <pinref part="GND2" gate="1" pin="GND"/>
-<wire x1="-7.62" y1="15.24" x2="-7.62" y2="10.16" width="0.1524" layer="91"/>
+<wire x1="-7.62" y1="15.24" x2="-7.62" y2="7.62" width="0.1524" layer="91"/>
+<wire x1="-7.62" y1="7.62" x2="-7.62" y2="5.08" width="0.1524" layer="91"/>
 <wire x1="-7.62" y1="15.24" x2="-7.62" y2="22.86" width="0.1524" layer="91"/>
 <junction x="-7.62" y="15.24"/>
@@
 <wire x1="-7.62" y1="22.86" x2="-25.4" y2="22.86" width="0.1524" layer="91"/>
 <pinref part="U1" gate="G$1" pin="1"/>
+<wire x1="-7.62" y1="7.62" x2="-15.24" y2="7.62" width="0.1524" layer="91"/>
+<junction x="-7.62" y="7.62"/>
+<pinref part="C1" gate="G$1" pin="2"/>
+<wire x1="-15.24" y1="7.62" x2="-15.24" y2="10.16" width="0.1524" layer="91"/>
 </segment>
 </net>
@@
 <segment>
 <pinref part="JP1" gate="A" pin="2"/>
-<wire x1="7.62" y1="45.72" x2="-5.08" y2="45.72" width="0.1524" layer="91"/>
+<wire x1="33.02" y1="45.72" x2="-5.08" y2="45.72" width="0.1524" layer="91"/>
 <wire x1="-5.08" y1="45.72" x2="-5.08" y2="96.52" width="0.1524" layer="91"/>
 <pinref part="U2" gate="G$1" pin="VDD"/>
-<wire x1="-5.08" y1="96.52" x2="22.86" y2="96.52" width="0.1524" layer="91"/>
+<wire x1="-5.08" y1="96.52" x2="15.24" y2="96.52" width="0.1524" layer="91"/>
 <label x="10.16" y="96.52" size="0.8128" layer="95"/>
 <pinref part="R1" gate="G$1" pin="2"/>
-<wire x1="22.86" y1="96.52" x2="35.56" y2="96.52" width="0.1524" layer="91"/>
+<wire x1="15.24" y1="96.52" x2="20.32" y2="96.52" width="0.1524" layer="91"/>
+<wire x1="20.32" y1="96.52" x2="35.56" y2="96.52" width="0.1524" layer="91"/>
 <wire x1="-12.7" y1="104.14" x2="-12.7" y2="106.68" width="0.1524" layer="91"/>
-<wire x1="-12.7" y1="106.68" x2="22.86" y2="106.68" width="0.1524" layer="91"/>
-<wire x1="22.86" y1="106.68" x2="22.86" y2="96.52" width="0.1524" layer="91"/>
-<junction x="22.86" y="96.52"/>
+<wire x1="-12.7" y1="106.68" x2="15.24" y2="106.68" width="0.1524" layer="91"/>
+<wire x1="15.24" y1="106.68" x2="15.24" y2="96.52" width="0.1524" layer="91"/>
+<junction x="15.24" y="96.52"/>
+<pinref part="C2" gate="G$1" pin="1"/>
+<wire x1="20.32" y1="88.9" x2="20.32" y2="96.52" width="0.1524" layer="91"/>
+<junction x="20.32" y="96.52"/>
 </segment>
 </net>
@@
 <pinref part="J1" gate="G$1" pin="4"/>
 <pinref part="JP1" gate="A" pin="4"/>
-<wire x1="-25.4" y1="50.8" x2="7.62" y2="50.8" width="0.1524" layer="91"/>
+<wire x1="-25.4" y1="50.8" x2="33.02" y2="50.8" width="0.1524" layer="91"/>
 </segment>
 </net>
@@
 <wire x1="2.54" y1="55.88" x2="2.54" y2="53.34" width="0.1524" layer="91"/>
 <pinref part="JP1" gate="A" pin="5"/>
-<wire x1="2.54" y1="53.34" x2="7.62" y2="53.34" width="0.1524" layer="91"/>
+<wire x1="2.54" y1="53.34" x2="33.02" y2="53.34" width="0.1524" layer="91"/>
 </segment>
 </net>
 <net name="N$8" class="1">
 <segment>
-<wire x1="-25.4" y1="12.7" x2="-12.7" y2="12.7" width="0.1524" layer="91"/>
-<wire x1="-12.7" y1="12.7" x2="-12.7" y2="20.32" width="0.1524" layer="91"/>
-<wire x1="-12.7" y1="20.32" x2="-2.54" y2="20.32" width="0.1524" layer="91"/>
+<wire x1="-25.4" y1="12.7" x2="-20.32" y2="12.7" width="0.1524" layer="91"/>
+<wire x1="-20.32" y1="12.7" x2="-20.32" y2="20.32" width="0.1524" layer="91"/>
+<wire x1="-20.32" y1="20.32" x2="-15.24" y2="20.32" width="0.1524" layer="91"/>
+<wire x1="-15.24" y1="20.32" x2="-2.54" y2="20.32" width="0.1524" layer="91"/>
 <wire x1="17.78" y1="20.32" x2="25.4" y2="20.32" width="0.1524" layer="91"/>
 <wire x1="25.4" y1="20.32" x2="25.4" y2="33.02" width="0.1524" layer="91"/>
-<wire x1="25.4" y1="33.02" x2="-12.7" y2="33.02" width="0.1524" layer="91"/>
-<wire x1="-12.7" y1="33.02" x2="-12.7" y2="20.32" width="0.1524" layer="91"/>
-<junction x="-12.7" y="20.32"/>
+<wire x1="25.4" y1="33.02" x2="-20.32" y2="33.02" width="0.1524" layer="91"/>
+<wire x1="-20.32" y1="33.02" x2="-20.32" y2="20.32" width="0.1524" layer="91"/>
+<junction x="-20.32" y="20.32"/>
 <pinref part="J2" gate="G$1" pin="1"/>
 <pinref part="U1" gate="G$1" pin="4"/>
 <pinref part="U1" gate="G$1" pin="3"/>
+<pinref part="C1" gate="G$1" pin="1"/>
+<wire x1="-15.24" y1="17.78" x2="-15.24" y2="20.32" width="0.1524" layer="91"/>
+<junction x="-15.24" y="20.32"/>
 </segment>
 </net>
@@
 <wire x1="25.4" y1="12.7" x2="25.4" y2="15.24" width="0.1524" layer="91"/>
 <pinref part="J2" gate="G$1" pin="2"/>
-<wire x1="-25.4" y1="15.24" x2="-17.78" y2="15.24" width="0.1524" layer="91"/>
-<wire x1="-17.78" y1="15.24" x2="-17.78" y2="2.54" width="0.1524" layer="91"/>
-<wire x1="-17.78" y1="2.54" x2="20.32" y2="2.54" width="0.1524" layer="91"/>
-<wire x1="20.32" y1="2.54" x2="20.32" y2="15.24" width="0.1524" layer="91"/>
+<wire x1="-25.4" y1="15.24" x2="-22.86" y2="15.24" width="0.1524" layer="91"/>
+<wire x1="-22.86" y1="15.24" x2="-22.86" y2="-2.54" width="0.1524" layer="91"/>
+<wire x1="-22.86" y1="-2.54" x2="20.32" y2="-2.54" width="0.1524" layer="91"/>
+<wire x1="20.32" y1="-2.54" x2="20.32" y2="15.24" width="0.1524" layer="91"/>
 <junction x="20.32" y="15.24"/>
 <pinref part="U1" gate="G$1" pin="2"/>
